File: cad/OpenCatFlap.kicad_sch (KiCad schematic)
At the start: 20 parts, among them P1 PIR Outside, P2 Flap IR Outside, P3 Flap IR Inside, P4 Servo Outside, P5 Servo Inside, P6 RFID Inside, P7 RFID Outside, P8 PIR Inside, U3 5V

Commit message: v2§
Parts:
- removed C4: 220uF, Capacitor_Tantalum_SMD:CP_EIA-7343-43_Kemet-X, symbol Device:C
- removed P1: PIR Outside, Connector_PinHeader_2.54mm:PinHeader_1x03_P2.54mm_Vertical, symbol OpenCatFlap:PIR Header
- added P1: IR Outside, Connector_PinHeader_2.54mm:PinHeader_1x04_P2.54mm_Vertical, symbol OpenCatFlap:IR_Barrier_Header
- added PIR_IN1: AMN33111, AMN33111_PAN, symbol OpenCatFlap:AMN33111
- added R10, R8: 10k, Resistor_SMD:R_0805_2012Metric, symbol Device:R
- added R6, R9: 200R, Resistor_SMD:R_0805_2012Metric, symbol Device:R
- added U1: TCRT5000L, TCRT5000_VIS, symbol OpenCatFlap:TCRT5000L
- P8: value PIR Inside -> PIR Outside
Connections:
- net at ArduinoESP32_L1.15 (Pin_15), C2.1, P2.1 (E+)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: now also C3.1, P1.1 (E+), P1.3 (D+), PIR_IN1.3 (VDD), U1.1 (C), U1.3 (A); no longer C3.2
- net at ArduinoESP32_L1.14 (Pin_14), C2.2, P4.2 (GND)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: now also C3.2, PIR_IN1.1 (GND), R10.2, R6.1, R8.1, R9.2; no longer C3.1
- net at ArduinoESP32_R1.10 (Pin_10), R7.1: now also PIR_IN1.2 (OUT); no longer P8.3 (In)
- net at ArduinoESP32_R1.7 (Pin_7): now also P1.4 (D-), R10.1
- net at ArduinoESP32_R1.8 (Pin_8): now also R8.2, U1.2 (E)
- net at ArduinoESP32_L1.10 (Pin_10), R2.2: now also P8.3 (In)
- new net: P1.2 (E-), R9.1
- new net: R6.2, U1.4 (C)
Other:
- moved on the sheet: C3

Commit message: board v2
Parts:
- P6, P7: footprint Connector_PinHeader_2.54mm:PinHeader_1x03_P2.54mm_Vertical -> Connector_PinHeader_2.54mm:PinHeader_1x04_P2.54mm_Vertical; symbol OpenCatFlap:PIR Header -> OpenCatFlap:RFID_Header
Connections:
- net at ArduinoESP32_L1.14 (Pin_14), C2.2, C3.2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: now also R1.2, R5.1
- net at P7.3 (In): now also ArduinoESP32_R1.3 (Pin_3); no longer ArduinoESP32_R1.14 (Pin_14)
- net at ArduinoESP32_R1.5 (Pin_5): now also P6.4 (RST)
- net at ArduinoESP32_R1.6 (Pin_6): now also P7.4 (RST)
- net at ArduinoESP32_R1.9 (Pin_9): now also P3.4 (D-), R1.1; no longer R1.2
- net at P2.4 (D-): now also ArduinoESP32_L1.9 (Pin_9), R5.2; no longer R5.1
Other:
- note added: "Reserved for TX1"
- note added: "Reserved for TX2"
- moved on the sheet: R1, R5

Commit message: update schematics
Parts:
- P8: Comment on the part (none) -> Currently using AMN31112. AMN41122 might be a better fit?
- PIR_IN1: Commen on part (none) -> Currently using AMN31112. AMN41122 might be a better fit?
Other:
- moved on the sheet: C2, P1, P2, P3, P4, P5, P6, P7, P8, R1, R10, R4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
