File: cad/OpenCatFlap.kicad_pcb (KiCad board)
At the start: 2 copper layers, 157 x 53 mm, 42 parts, among them P1 Outside PIR, P2 IR Barrier Outside, P3 IR Barrier Inside, P4 Servo Outside, P5 Servo Inside, U1 DOIT-ESP32-DEVKIT-V1, U2 AMN33111, U3 5V, U4 TMS3705DDRQ1, U7 TMS3705DDRQ1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

Commit message: Revert "meow"
This reverts commit 70150f40207d0a9de3da7c8185f4e8c8306b4b66.
Parts:
- removed C10, C11, C12, C9: 10pF, Capacitor_SMD:C_0805_2012Metric
- removed C2: 100nF, Capacitor_SMD:C_0805_2012Metric
- removed C3: 22uF, Capacitor_SMD:CP_Elec_8x10
- removed C4, C7, C8: 220pF, Capacitor_SMD:C_0805_2012Metric
- removed C5, C6: 3.3nF, Capacitor_SMD:C_0805_2012Metric
- removed R10, R11, R14, R15: 4.7, Resistor_SMD:R_0805_2012Metric
- removed R12, R9: 150k, Resistor_SMD:R_0805_2012Metric
- removed R13, R8: 47k, Resistor_SMD:R_0805_2012Metric
- removed R16, R7: 220, Resistor_SMD:R_0805_2012Metric
- removed U4, U7: TMS3705DDRQ1, OpenCatFlap:D16
- removed U5, U6: ~, OpenCatFlap:Power Header
- removed Y1, Y2: Crystal 4MHz, Crystal:Crystal_HC49-4H_Vertical
- added P6: RFID inside, OpenCatFlap:PIR Header, F.Cu at (177.6, 109.1)
- added P7: RFID outside, OpenCatFlap:PIR Header, F.Cu at (134.4, 109.1)
- C1: value 220pF -> 220uF; footprint Capacitor_SMD:C_0805_2012Metric -> Capacitor_THT:CP_Radial_D5.0mm_P2.50mm
- R4, R5: moved to F.Cu
- moved P1 32.8 mm to (182.9, 73.7)
- moved P2 31.9 mm to (182.9, 76.2)
- moved P4 31.9 mm to (182.9, 91.4)
- moved U1 30.8 mm to (139.7, 78.7)
- moved R3 28.4 mm to (179.2, 68.5)
- moved R1 27.4 mm to (179.2, 78.6)
- moved R6 27.3 mm to (179.2, 83.8)
- moved R5 23.4 mm to (106.4, 99.0), turned to -90 degrees
- moved P3 23.1 mm to (94.0, 109.1)
- moved P5 22.9 mm to (109.0, 109.1)
- moved R4 21.8 mm to (100.4, 96.4)
- moved C1 20.2 mm to (131.8, 99.0), turned to -90 degrees
- moved U3 19.3 mm to (136.9, 101.5), turned to 180 degrees
- moved R2 5.08 mm to (147.1, 99.0)
Connections:
- C1 pad 1: Net-(U5-GND) -> GND
- C1 pad 2: GND -> +5V
- U1 pad 14: Net-(U1-GPIO9_SHD/SD2) -> unconnected-(U1-GPIO9_SHD/SD2-Pad14)
- U1 pad 35: Net-(U1-GPIO22_I2C-SCL) -> unconnected-(U1-GPIO22_I2C-SCL-Pad35)
Routing:
- net +5V: track 380.5 -> 200.4 mm, vias 4 -> 0
- net GND: track 412.7 -> 268.8 mm, vias 0 -> 2
- net Net-(P4-PWM): track 186.5 -> 86.6 mm, vias 1 -> 0
- net Net-(U1-GPIO22_I2C-SCL): track 96.8 -> 0.00 mm, vias 2 -> 0
- net Net-(P1-In): track 160.2 -> 67.8 mm, vias 0 -> 1
- net Net-(U1-GPIO9_SHD/SD2): track 73.0 -> 0.00 mm, vias 2 -> 0
- net Net-(P2-D-): track 134.5 -> 62.2 mm, vias 0 -> 1
- net Net-(P7-In): track 85.3 -> 17.8 mm
- net Net-(P6-In): track 6.43 -> 71.9 mm, vias 0 -> 1
- net Net-(U4-SCIO): track 55.6 -> 0.00 mm, vias 1 -> 0
- net Net-(U1-GPIO27_ADC2-CH7_RTC-GPIO17): track 94.6 -> 60.8 mm, vias 0 -> 1
- net Net-(U7-OSC2): track 30.9 -> 0.00 mm
- net Net-(U4-OSC2): track 29.7 -> 0.00 mm
- net Net-(P3-D-): track 54.1 -> 82.1 mm, vias 1 -> 2
- net Net-(U4-OSC1): track 25.2 -> 0.00 mm
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Other:
- board size 157 x 53 mm -> 97 x 53 mm

Commit message: boop
Parts:
- removed C1: 220uF, Capacitor_THT:CP_Radial_D5.0mm_P2.50mm
- removed R6: 100R, Resistor_SMD:R_0805_2012Metric
- removed U1: DOIT-ESP32-DEVKIT-V1, OpenCatFlap:ESP32-DOIT-DEVKIT
- removed U2: AMN33111, OpenCatFlap:AMN33111_PAN
- added ArduinoESP32_L1: VIN-D13, Connector_PinHeader_2.54mm:PinHeader_1x15_P2.54mm_Vertical, F.Cu at (93.7, 83.7)
- added ArduinoESP32_R1: Pin TX1-D12, Connector_PinHeader_2.54mm:PinHeader_1x15_P2.54mm_Vertical, F.Cu at (94.4, 68.5)
- added C2: C_Polarized, Capacitor_SMD:CP_Elec_8x10, F.Cu at (139.5, 65.9)
- added C3: C_Polarized, Capacitor_SMD:CP_Elec_8x10, F.Cu at (139.5, 88.8)
- added C4: 220uF, Capacitor_Tantalum_SMD:CP_EIA-7343-43_Kemet-X, F.Cu at (138.9, 76.1)
- added P8: PIR Inside, Connector_PinHeader_2.54mm:PinHeader_1x03_P2.54mm_Vertical, F.Cu at (121.7, 60.9)
- added R7: 100k, Resistor_SMD:R_0805_2012Metric, F.Cu at (125.8, 73.6)
- P1: value Outside PIR -> PIR Outside; footprint OpenCatFlap:PIR Header -> Connector_PinHeader_2.54mm:PinHeader_1x03_P2.54mm_Vertical
- P2: value IR Barrier Outside -> Flap IR Outside; footprint OpenCatFlap:IR Barrier Header -> Connector_PinHeader_2.54mm:PinHeader_1x04_P2.54mm_Vertical
- P3: value IR Barrier Inside -> Flap IR Inside; footprint OpenCatFlap:IR Barrier Header -> Connector_PinHeader_2.54mm:PinHeader_1x04_P2.54mm_Vertical
- P4, P5: footprint OpenCatFlap:Servo Header -> Connector_PinHeader_2.54mm:PinHeader_1x03_P2.54mm_Vertical
- P6: value RFID inside -> RFID Inside; footprint OpenCatFlap:PIR Header -> Connector_PinHeader_2.54mm:PinHeader_1x03_P2.54mm_Vertical
- P7: value RFID outside -> RFID Outside; footprint OpenCatFlap:PIR Header -> Connector_PinHeader_2.54mm:PinHeader_1x03_P2.54mm_Vertical
- R1, R4, R5: moved to B.Cu
- R3: value 100k -> 100R; moved to B.Cu
- U3: footprint OpenCatFlap:Power Header -> Connector_PinHeader_2.54mm:PinHeader_1x02_P2.54mm_Vertical
- moved P6 92.4 mm to (98.8, 60.9), turned to -90 degrees
- moved R1 76.6 mm to (103.9, 64.3), turned to -90 degrees
- moved P2 73.5 mm to (111.5, 93.9), turned to -90 degrees
- moved R3 73.3 mm to (109.0, 89.7), turned to 90 degrees
- moved P1 64.5 mm to (121.7, 93.9), turned to -90 degrees
- moved P5 53.4 mm to (131.8, 60.9), turned to -90 degrees
- moved P3 51.3 mm to (111.5, 60.9), turned to -90 degrees
- moved P4 51.1 mm to (131.8, 93.9), turned to -90 degrees
- moved P7 38.7 mm to (98.8, 93.9), turned to -90 degrees
- moved R4 33.2 mm to (109.0, 64.3), turned to 90 degrees
- moved R2 29.4 mm to (125.8, 78.6), turned to 180 degrees
- moved U3 20.9 mm to (142.0, 81.2), turned to -90 degrees
- moved R5 8.90 mm to (103.9, 90.4), turned to 90 degrees
Connections:
- net +5V renamed Net-(ArduinoESP32_L1-Pin_15)
- P1 pad 2: GND -> Net-(ArduinoESP32_L1-Pin_14)
- P1 pad 3: Net-(P1-In) -> Net-(ArduinoESP32_L1-Pin_10)
- P4 pad 2: GND -> Net-(ArduinoESP32_L1-Pin_14)
- P5 pad 2: GND -> Net-(ArduinoESP32_L1-Pin_14)
- P6 pad 2: GND -> Net-(ArduinoESP32_L1-Pin_14)
- P7 pad 2: GND -> Net-(ArduinoESP32_L1-Pin_14)
- R1 pad 1: GND -> Net-(P3-D-)
- R1 pad 2: Net-(P2-E-) -> Net-(ArduinoESP32_R1-Pin_9)
- R2 pad 1: GND -> Net-(ArduinoESP32_L1-Pin_14)
- R2 pad 2: Net-(U1-GPIO27_ADC2-CH7_RTC-GPIO17) -> Net-(ArduinoESP32_L1-Pin_10)
- R3 pad 1: GND -> Net-(P2-E-)
- R3 pad 2: Net-(P1-In) -> Net-(ArduinoESP32_L1-Pin_14)
- R4 pad 1: GND -> Net-(ArduinoESP32_L1-Pin_14)
- R5 pad 1: GND -> Net-(P2-D-)
- R5 pad 2: Net-(P3-D-) -> Net-(ArduinoESP32_L1-Pin_9)
- U3 pad 2: GND -> Net-(ArduinoESP32_L1-Pin_14)
Routing:
- net GND: track 268.8 -> 0.00 mm, vias 2 -> 0
- net Net-(ArduinoESP32_L1-Pin_14): track 0.00 -> 170.6 mm, vias 0 -> 1
- net Net-(P3-D-): track 82.1 -> 2.54 mm, vias 2 -> 0
- net Net-(ArduinoESP32_L1-Pin_15): track 200.4 -> 126.7 mm
- net Net-(ArduinoESP32_L1-Pin_11): track 86.6 -> 13.3 mm
- net Net-(P1-In): track 67.8 -> 0.00 mm, vias 1 -> 0
- net Net-(U1-GPIO27_ADC2-CH7_RTC-GPIO17): track 60.8 -> 0.00 mm, vias 1 -> 0
- net Net-(ArduinoESP32_R1-Pin_4): track 71.9 -> 12.0 mm, vias 1 -> 0
- net Net-(P2-D-): track 62.2 -> 2.54 mm, vias 1 -> 0
- net Net-(ArduinoESP32_R1-Pin_11): track 46.1 -> 10.5 mm
- net Net-(ArduinoESP32_R1-Pin_14): track 17.8 -> 44.7 mm
- net Net-(ArduinoESP32_L1-Pin_10): track 0.00 -> 20.6 mm
- net Net-(ArduinoESP32_R1-Pin_10): track 0.00 -> 17.7 mm
- net Net-(ArduinoESP32_L1-Pin_9): track 0.00 -> 12.6 mm
- net Net-(ArduinoESP32_R1-Pin_9): track 0.00 -> 12.1 mm
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Other:
- board size 97 x 53 mm -> 53.3 x 38.1 mm
- board text added: "+"
- board text added: "GND"
