File: cad/OpenCatFlap.kicad_pcb (KiCad board)
At the start: 2 copper layers, 53.3 x 38.1 mm, 20 parts, among them P1 PIR Outside, P2 Flap IR Outside, P3 Flap IR Inside, P4 Servo Outside, P5 Servo Inside, P6 RFID Inside, P7 RFID Outside, P8 PIR Inside, U3 5V

Commit message: Fix wiring
Routing:
- net Net-(ArduinoESP32_L1-Pin_14): track 170.6 -> 167.1 mm
Other:
- board text added: "1000uF"
Changed lines of the file:
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@@
       (outputformat 1)
       (mirror false)
-      (drillshape 1)
+      (drillshape 0)
       (scaleselection 1)
-      (outputdirectory "")
+      (outputdirectory "./gbr")
     )
   )
@@
     (fp_line (start 1 0.625) (end -1 0.625)
       (stroke (width 0.1) (type solid)) (layer "F.Fab"))
-    (pad "1" smd roundrect (at -0.9125 0) (size 1.025 1.4) (layers "F.Cu" "F.Paste" "F.Mask") (roundrect_rratio 0.243902)
+    (pad "1" smd roundrect (at -0.9125 0) (size 1.025 1.4) (layers "F.Cu" "F.Paste" "F.Mask") (roundrect_rratio 0.243902439)
       (net 29 "Net-(ArduinoESP32_R1-Pin_10)") (pintype "passive"))
-    (pad "2" smd roundrect (at 0.9125 0) (size 1.025 1.4) (layers "F.Cu" "F.Paste" "F.Mask") (roundrect_rratio 0.243902)
+    (pad "2" smd roundrect (at 0.9125 0) (size 1.025 1.4) (layers "F.Cu" "F.Paste" "F.Mask") (roundrect_rratio 0.243902439)
       (net 18 "Net-(ArduinoESP32_L1-Pin_14)") (pintype "passive"))
     (model "${KICAD6_3DMODEL_DIR}/Resistor_SMD.3dshapes/R_0805_2012Metric.wrl"
@@
     (fp_line (start 1 0.625) (end -1 0.625)
       (stroke (width 0.1) (type solid)) (layer "F.Fab"))
-    (pad "1" smd roundrect (at -0.9125 0 180) (size 1.025 1.4) (layers "F.Cu" "F.Paste" "F.Mask") (roundrect_rratio 0.243902)
+    (pad "1" smd roundrect (at -0.9125 0 180) (size 1.025 1.4) (layers "F.Cu" "F.Paste" "F.Mask") (roundrect_rratio 0.243902439)
       (net 18 "Net-(ArduinoESP32_L1-Pin_14)") (pintype "passive"))
-    (pad "2" smd roundrect (at 0.9125 0 180) (size 1.025 1.4) (layers "F.Cu" "F.Paste" "F.Mask") (roundrect_rratio 0.243902)
+    (pad "2" smd roundrect (at 0.9125 0 180) (size 1.025 1.4) (layers "F.Cu" "F.Paste" "F.Mask") (roundrect_rratio 0.243902439)
       (net 14 "Net-(ArduinoESP32_L1-Pin_10)") (pintype "passive"))
     (model "${KICAD6_3DMODEL_DIR}/Resistor_SMD.3dshapes/R_0805_2012Metric.wrl"
@@
     (fp_line (start 3.65 2.15) (end 3.65 -2.15)
       (stroke (width 0.1) (type solid)) (layer "F.Fab"))
-    (pad "1" smd roundrect (at -3.1125 0 180) (size 2.075 2.55) (layers "F.Cu" "F.Paste" "F.Mask") (roundrect_rratio 0.120482)
+    (pad "1" smd roundrect (at -3.1125 0 180) (size 2.075 2.55) (layers "F.Cu" "F.Paste" "F.Mask") (roundrect_rratio 0.1204819277)
       (net 19 "Net-(ArduinoESP32_L1-Pin_15)") (pintype "passive"))
-    (pad "2" smd roundrect (at 3.1125 0 180) (size 2.075 2.55) (layers "F.Cu" "F.Paste" "F.Mask") (roundrect_rratio 0.120482)
+    (pad "2" smd roundrect (at 3.1125 0 180) (size 2.075 2.55) (layers "F.Cu" "F.Paste" "F.Mask") (roundrect_rratio 0.1204819277)
       (net 18 "Net-(ArduinoESP32_L1-Pin_14)") (pintype "passive"))
     (model "${KICAD6_3DMODEL_DIR}/Capacitor_Tantalum_SMD.3dshapes/CP_EIA-7343-43_Kemet-X.wrl"
@@
     (fp_line (start 1 0.625) (end 1 -0.625)
       (stroke (width 0.1) (type solid)) (layer "B.Fab"))
-    (pad "1" smd roundrect (at -0.9125 0 90) (size 1.025 1.4) (layers "B.Cu" "B.Paste" "B.Mask") (roundrect_rratio 0.243902)
+    (pad "1" smd roundrect (at -0.9125 0 90) (size 1.025 1.4) (layers "B.Cu" "B.Paste" "B.Mask") (roundrect_rratio 0.243902439)
       (net 5 "Net-(P2-D-)") (pintype "passive"))
-    (pad "2" smd roundrect (at 0.9125 0 90) (size 1.025 1.4) (layers "B.Cu" "B.Paste" "B.Mask") (roundrect_rratio 0.243902)
+    (pad "2" smd roundrect (at 0.9125 0 90) (size 1.025 1.4) (layers "B.Cu" "B.Paste" "B.Mask") (roundrect_rratio 0.243902439)
       (net 13 "Net-(ArduinoESP32_L1-Pin_9)") (pintype "passive"))
     (model "${KICAD6_3DMODEL_DIR}/Resistor_SMD.3dshapes/R_0805_2012Metric.wrl"
@@
     (fp_line (start 1 0.625) (end 1 -0.625)
       (stroke (width 0.1) (type solid)) (layer "B.Fab"))
-    (pad "1" smd roundrect (at -0.9125 0 270) (size 1.025 1.4) (layers "B.Cu" "B.Paste" "B.Mask") (roundrect_rratio 0.243902)
+    (pad "1" smd roundrect (at -0.9125 0 270) (size 1.025 1.4) (layers "B.Cu" "B.Paste" "B.Mask") (roundrect_rratio 0.243902439)
       (net 7 "Net-(P3-D-)") (pintype "passive"))
-    (pad "2" smd roundrect (at 0.9125 0 270) (size 1.025 1.4) (layers "B.Cu" "B.Paste" "B.Mask") (roundrect_rratio 0.243902)
+    (pad "2" smd roundrect (at 0.9125 0 270) (size 1.025 1.4) (layers "B.Cu" "B.Paste" "B.Mask") (roundrect_rratio 0.243902439)
       (net 28 "Net-(ArduinoESP32_R1-Pin_9)") (pintype "passive"))
     (model "${KICAD6_3DMODEL_DIR}/Resistor_SMD.3dshapes/R_0805_2012Metric.wrl"
@@
     (fp_line (start 1 0.625) (end 1 -0.625)
       (stroke (width 0.1) (type solid)) (layer "B.Fab"))
-    (pad "1" smd roundrect (at -0.9125 0 90) (size 1.025 1.4) (layers "B.Cu" "B.Paste" "B.Mask") (roundrect_rratio 0.243902)
+    (pad "1" smd roundrect (at -0.9125 0 90) (size 1.025 1.4) (layers "B.Cu" "B.Paste" "B.Mask") (roundrect_rratio 0.243902439)
       (net 18 "Net-(ArduinoESP32_L1-Pin_14)") (pintype "passive"))
-    (pad "2" smd roundrect (at 0.9125 0 90) (size 1.025 1.4) (layers "B.Cu" "B.Paste" "B.Mask") (roundrect_rratio 0.243902)
+    (pad "2" smd roundrect (at 0.9125 0 90) (size 1.025 1.4) (layers "B.Cu" "B.Paste" "B.Mask") (roundrect_rratio 0.243902439)
       (net 6 "Net-(P3-E-)") (pintype "passive"))
     (model "${KICAD6_3DMODEL_DIR}/Resistor_SMD.3dshapes/R_0805_2012Metric.wrl"
@@
     (fp_line (start 1 0.625) (end 1 -0.625)
       (stroke (width 0.1) (type solid)) (layer "B.Fab"))
-    (pad "1" smd roundrect (at -0.9125 0 90) (size 1.025 1.4) (layers "B.Cu" "B.Paste" "B.Mask") (roundrect_rratio 0.243902)
+    (pad "1" smd roundrect (at -0.9125 0 90) (size 1.025 1.4) (layers "B.Cu" "B.Paste" "B.Mask") (roundrect_rratio 0.243902439)
       (net 4 "Net-(P2-E-)") (pintype "passive"))
-    (pad "2" smd roundrect (at 0.9125 0 90) (size 1.025 1.4) (layers "B.Cu" "B.Paste" "B.Mask") (roundrect_rratio 0.243902)
+    (pad "2" smd roundrect (at 0.9125 0 90) (size 1.025 1.4) (layers "B.Cu" "B.Paste" "B.Mask") (roundrect_rratio 0.243902439)
       (net 18 "Net-(ArduinoESP32_L1-Pin_14)") (pintype "passive"))
     (model "${KICAD6_3DMODEL_DIR}/Resistor_SMD.3dshapes/R_0805_2012Metric.wrl"
@@
   (gr_text "+" (at 101.36 58.32 180) (layer "F.SilkS")
     (effects (font (size 1 1) (thickness 0.15)) (justify left bottom))
+  )
+  (gr_text "1000uF\n" (at 139.46 65.94) (layer "F.SilkS")
+    (effects (font (size 1 1) (thickness 0.15)))
+  )
+  (gr_text "1000uF" (at 139.46 88.8) (layer "F.SilkS")
+    (effects (font (size 1 1) (thickness 0.15)))
   )
   (gr_text "+" (at 124.22 58.32 180) (layer "F.SilkS")
@@
   (segment (start 139.46 81.18) (end 139.46 79.785) (width 0.25) (layer "F.Cu") (net 18))
   (segment (start 139.46 76.1) (end 139.46 69.19) (width 0.25) (layer "F.Cu") (net 18))
-  (segment (start 139.46 72.923604) (end 127.396396 60.86) (width 0.25) (layer "F.Cu") (net 18))
   (segment (start 139.46 81.18) (end 129.305 81.18) (width 0.25) (layer "F.Cu") (net 18))
   (segment (start 139.46 92.05) (end 139.46 88.8) (width 0.25) (layer "F.Cu") (net 18))
@@
   (segment (start 139.46 81.18) (end 139.46 72.923604) (width 0.25) (layer "F.Cu") (net 18))
   (segment (start 126.76 78.64) (end 129.3025 81.1825) (width 0.25) (layer "F.Cu") (net 18))
+  (segment (start 137.63 69.19) (end 139.46 69.19) (width 0.25) (layer "F.Cu") (net 18))
+  (segment (start 129.3 60.86) (end 137.63 69.19) (width 0.25) (layer "F.Cu") (net 18))
   (segment (start 129.305 81.18) (end 129.3025 81.1825) (width 0.25) (layer "F.Cu") (net 18))
   (segment (start 126.765 83.72) (end 126.765 91.345) (width 0.25) (layer "F.Cu") (net 18))
@@
   (segment (start 124.22 88.8) (end 126.765 86.255) (width 0.25) (layer "B.Cu") (net 18))
   (segment (start 107.9925 64.2375) (end 108.98 65.225) (width 0.25) (layer "B.Cu") (net 18))
+  (segment (start 128.125 62.035) (end 129.3 60.86) (width 0.25) (layer "B.Cu") (net 18))
   (segment (start 107.4275 90.3525) (end 108.98 88.8) (width 0.25) (layer "B.Cu") (net 18))
   (segment (start 119.14 60.86) (end 114.775 65.225) (width 0.25) (layer "B.Cu") (net 18))
@@
   (segment (start 96.28 93.88) (end 99.8075 90.3525) (width 0.25) (layer "B.Cu") (net 18))
   (segment (start 108.98 88.8) (end 124.22 88.8) (width 0.25) (layer "B.Cu") (net 18))
-  (segment (start 129.3 60.86) (end 128.125 62.035) (width 0.25) (layer "B.Cu") (net 18))
   (segment (start 128.125 62.035) (end 120.315 62.035) (width 0.25) (layer "B.Cu") (net 18))
   (segment (start 114.775 65.225) (end 108.98 65.225) (width 0.25) (layer "B.Cu") (net 18))
