File: cad/opencatflap/opencatflap.kicad_sch (KiCad schematic)
At the start: 61 parts, among them J1 Screw_Terminal_01x02, J2 Screw_Terminal_01x04, J3 Screw_Terminal_01x01, P1 PIR Outside, P10 RFID OutSide, P11 Servo Inside, P12 Servo Outside, P2 Flap IR Inside, P4 Flap IR Outside, P9 RFID Inside, Q1 BSS138, Q2 BSS138, Q3 BSS138, Q4 BSS138, Q5 BC546B, Q6 BC546B, U1 TPS22810DRV, U2 TPS22810DRV, U3 LM1117DT-3.3, U4 LM324, U5 TCRT5000L, U6 LMR54410DBVR, U7 AMN33111

Commit message: update
Parts:
- removed ArduinoESP32_L1: VIN-D13, Connector_PinHeader_2.54mm:PinHeader_1x15_P2.54mm_Vertical, symbol Connector:Conn_01x15_Pin
- removed ArduinoESP32_R1: Pin TX1-D12, Connector_PinHeader_2.54mm:PinHeader_1x15_P2.54mm_Vertical, symbol Connector:Conn_01x15_Pin
- removed C1, C2: 10u, Capacitor_SMD:C_0805_2012Metric, symbol Device:C_Small
- removed C10, C6: 100n, Capacitor_SMD:C_0603_1608Metric, symbol Device:C
- removed C3: 100n, Capacitor_SMD:C_0402_1005Metric, symbol Device:C
- removed C4: 4.7u, Capacitor_SMD:C_1210_3225Metric, symbol Device:C
- removed C5, C7: 10u, Capacitor_SMD:C_0805_2012Metric, symbol Device:C
- removed C8, C9: 100u, Capacitor_SMD:CP_Elec_6.3x7.7, symbol Device:C_Polarized_US
- removed J1: Screw_Terminal_01x02, TerminalBlock_4Ucon:TerminalBlock_4Ucon_1x02_P3.50mm_Vertical, symbol Connector:Screw_Terminal_01x02
- removed J2: Screw_Terminal_01x04, Connector_PinHeader_2.54mm:PinHeader_1x04_P2.54mm_Vertical, symbol Connector:Screw_Terminal_01x04
- removed J3: Screw_Terminal_01x01, Connector_PinHeader_2.54mm:PinHeader_1x01_P2.54mm_Vertical, symbol Connector:Screw_Terminal_01x01
- removed L1: 12u, Alexander Project1:SDR0805120ML, symbol Device:L
- removed P1: PIR Outside, Connector_PinHeader_2.54mm:PinHeader_1x03_P2.54mm_Vertical, symbol OpenCatFlap:PIR Header
- removed P10: RFID OutSide, Connector_PinHeader_2.54mm:PinHeader_1x04_P2.54mm_Vertical, symbol OpenCatFlap:RFID_Header
- removed P11: Servo Inside, Connector_PinHeader_2.54mm:PinHeader_1x03_P2.54mm_Vertical, symbol OpenCatFlap:Servo_Header
- removed P12: Servo Outside, Connector_PinHeader_2.54mm:PinHeader_1x03_P2.54mm_Vertical, symbol OpenCatFlap:Servo_Header
- removed P2: Flap IR Inside, Connector_PinHeader_2.54mm:PinHeader_1x04_P2.54mm_Vertical, symbol OpenCatFlap:IR_Barrier_Header
- removed P4: Flap IR Outside, Connector_PinHeader_2.54mm:PinHeader_1x04_P2.54mm_Vertical, symbol OpenCatFlap:IR_Barrier_Header
- removed P9: RFID Inside, Connector_PinHeader_2.54mm:PinHeader_1x04_P2.54mm_Vertical, symbol OpenCatFlap:RFID_Header
- removed Q1, Q2, Q3, Q4: BSS138, Package_TO_SOT_SMD:SOT-23, symbol Transistor_FET:BSS138
- removed Q5, Q6: BC546B, Package_TO_SOT_THT:TO-92_Inline, symbol Transistor_BJT:BC546
- removed R1: 200R, Resistor_SMD:R_0603_1608Metric, symbol Device:R
- removed R10: 118k, Resistor_SMD:R_0402_1005Metric, symbol Device:R
- removed R11, R12, R13, R14, R15, R16, R18, R20, R4, R6: 10k, Resistor_SMD:R_0603_1608Metric, symbol Device:R_Small
- removed R2, R7, R8, R9: 33k, Resistor_SMD:R_0603_1608Metric, symbol Device:R
- removed R21, R5: 566R, Resistor_SMD:R_0603_1608Metric, symbol Device:R
- removed R22, R24, R25, R3: 10k, Resistor_SMD:R_0603_1608Metric, symbol Device:R
- removed R23: 22.1k, Resistor_SMD:R_0402_1005Metric, symbol Device:R
- removed RV1: 10k, Alexander Project1:3296W-1, symbol Device:R_Potentiometer
- removed U1, U2: TPS22810DRV, Package_SON:WSON-6-1EP_2x2mm_P0.65mm_EP1x1.6mm, symbol Power_Management:TPS22810DRV
- removed U3: LM1117DT-3.3, Package_TO_SOT_SMD:TO-252-3_TabPin2, symbol Regulator_Linear:LM1117DT-3.3
- removed U4: LM324, Alexander Project1:SOIC127P600X175-14N, symbol Amplifier_Operational:LM324
- removed U5: TCRT5000L, Alexander Project1:TCRT5000L, symbol OpenCatFlap:TCRT5000L
- removed U6: LMR54410DBVR, Alexander Project1:LMR54410DBVR, symbol Bottom-A-2nd-Varient:LMR54410DBVR
- removed U7: AMN33111, AMN33111, symbol Alexander Project1:AMN-33111
- added C1, C2, C4, C5: 10uF, OpenCatFlap:CAP_CL31A_SAM, symbol OpenCatFlap:C_CL31A106MBHNNNE
- added C10: 100uF, Capacitor_SMD:CP_Elec_6.3x7.7, symbol VH1E101ME077000CE0_1
- added C11, C12, C31, C32, C37, C40: 1nF, Capacitor_SMD:C_0603_1608Metric, symbol OpenCatFlap:C_CC0603JRX7R9BB102
- added C13, C14, C29, C30: 22pF, Capacitor_SMD:C_0603_1608Metric, symbol OpenCatFlap:C_0603CG220J500NT
- added C15: 1.5nF, Capacitor_SMD:C_0603_1608Metric, symbol 0603B152J500CT
- added C16, C17, C18, C19, C24, C25, C26, C27: 100nF, Capacitor_SMD:C_0603_1608Metric, symbol OpenCatFlap:C_CC0603KRX7R7BB104
- added C20, C21, C22, C23, C36, C39: 10nF, Capacitor_SMD:C_0603_1608Metric, symbol OpenCatFlap:C_CC0603KRX7R7BB103
- added C28: 1.5nF, Capacitor_SMD:C_0603_1608Metric, symbol 0603B152J500CT_1
- added C3, C6: 100nF, Capacitor_SMD:C_1210_3225Metric, symbol OpenCatFlap:C_CC1210KKX7R0BB104
- added C33, C8: 12pF - 60 pF, OpenCatFlap:VCAP_GKGXXX15_SGM, symbol OpenCatFlap:C_GKG60015
- added C7: 4.7uF, Capacitor_SMD:C_1206_3216Metric, symbol CGA5L1X8R1E475KT0Y0N
- added C9: 100uF, Capacitor_SMD:CP_Elec_6.3x7.7, symbol VH1E101ME077000CE0
- added L1: 12uH, OpenCatFlap:LBM2016TI20J, symbol LBM2016T120J
- added P1, P11, P7, P8: S2B-PH-K-SLFSN, OpenCatFlap:CONN_S2B-PH-K-S_JST, symbol OpenCatFlap:S2B-PH-K-SLFSN
- added P10: IL-G-2P-S3T2-SA, OpenCatFlap:CONN_S2B-PH-K-S_JST, symbol OpenCatFlap:S2B-PH-K-SLFSN
- added P12, P4, P5, P6, P9: S3B-PH-K-S LFSN, OpenCatFlap:CONN_S3B-PH-K-S_JST, symbol OpenCatFlap:S3B-PH-K-S_LFSN
- added P2, P3: S4B-PH-K-S_LF__SN_, OpenCatFlap:CONN_S4B-PH-K-S_JST, symbol OpenCatFlap:S4B-PH-K-S_LFSN
- added Q1: BSS138L, OpenCatFlap:BSS138L, symbol BSS138L
- added Q2: BSS138L, OpenCatFlap:BSS138L, symbol BSS138L_1
- added Q3: BSS138L, OpenCatFlap:BSS138L, symbol BSS138L_2
- added Q4: BSS138L, OpenCatFlap:BSS138L, symbol BSS138L_3
- added R1: 118kΩ, Resistor_SMD:R_0603_1608Metric, symbol ERJ3EKF1183V
- added R10, R11, R14, R15, R3, R4, R5, R6, R7, R8, R9: 10kΩ, Resistor_SMD:R_0603_1608Metric, symbol OpenCatFlap:R_RC0603FR-0710KL
- added R12, R23, R32: 10k, Resistor_SMD:R_0603_1608Metric, symbol OpenCatFlap:R_RC0603FR-0710KL
- added R13: 560Ω, Resistor_SMD:R_0603_1608Metric, symbol RC0603FR-07560RL
- added R16: 560Ω, Resistor_SMD:R_0603_1608Metric, symbol RC0603FR-07560RL_1
- added R17, R18, R19, R20, R24, R25: 33kΩ, Resistor_SMD:R_0603_1608Metric, symbol OpenCatFlap:R_RC0603FR-0733KL
- added R2: 22.1kΩ, Resistor_SMD:R_0603_1608Metric, symbol RNCF0603BKC22K1
- added R21: 27Ω, Resistor_SMD:R_0603_1608Metric, symbol RC0603FR-0727RL
- added R22: 27Ω, Resistor_SMD:R_0603_1608Metric, symbol RC0603FR-0727RL_1
- added R27: 11.2k, Resistor_SMD:R_0603_1608Metric, symbol Device:R
- added R28, R31: 82, Resistor_SMD:R_0603_1608Metric, symbol Device:R
- added R29: 4.7k, Resistor_SMD:R_0603_1608Metric, symbol Device:R
- added R30: 16.5k, Resistor_SMD:R_0603_1608Metric, symbol Device:R
- added U1: ARDUINO_NANO, OpenCatFlap:Arduino Nano ESP32, symbol ARDUINO_NANO
- added U10: SENSOR MOTION SPOT 5V BLK LENS, OpenCatFlap:AMN33111, symbol SENSOR MOTION SPOT 5V BLK LENS
- added U11: EM4095, OpenCatFlap:EM4095, symbol EM4095
- added U12: EM4095, OpenCatFlap:EM4095, symbol EM4095_1
- added U13, U5: NE555D, Package_SO:SOIC-8_3.9x4.9mm_P1.27mm, symbol Timer:NE555D
- added U14, U4, U9: BC546BBK, Package_TO_SOT_THT:TO-92L_Inline, symbol BC546BBK_1
- added U2: LM1117DTX-3.3/NOPB, OpenCatFlap:LM1117DTX-3.3NOPB, symbol OpenCatFlap:LM1117DTX-3.3_NOPB
- added U3: LMR54410DBVR, OpenCatFlap:U_SOT-23_TEX, symbol LMR54410DBVR
- added U6: TPS22810DRVR, OpenCatFlap:DRV0006A_NV, symbol TPS22810DRVR
- added U7: TPS22810DRVR, OpenCatFlap:DRV0006A_NV, symbol TPS22810DRVR_1
- added U8: BC546BBK, Package_TO_SOT_THT:TO-92L_Inline, symbol BC546BBK
- R26: value 200R -> 3.3k; Manufacturer (none) -> YAGEO; Manufacturer Part (none) -> AC0603FR-073K3L
Connections:
- net +3V3: now also C2.1, P12.1, P2.3, P3.3, P6.1, P9.1, Q1.1 (G), Q2.1 (G), Q3.1 (G), Q4.1 (G), R12.2, R13.1, R16.1, R3.2, R4.2, R5.2, R8.2, R9.2, U10.1, U2.4 (OUT)
- net +5V: now also C1.1, C10.1, C16.1, C27.1, C4.1, C5.1, C9.1, L1.2, P4.1, P5.1, R1.2, R10.2, R11.2, R6.2, R7.2, U11.4, U11.7, U12.4, U12.7, U2.3 (INPUT), U6.6 (VIN), U7.6 (VIN)
- net +9V: now also R26.2, C6.2, C7.2, P1.1, R29.2, U1.30 (VIN), U13.4 (R), U13.8 (VCC), U3.4 (EN), U3.5 (VIN), U5.4 (R), U5.8 (VCC)
- net Flap_IR_Inside: now also P2.4, R14.1, U1.12 (D9)
- net Flap_IR_Outside: now also P3.4, R15.1, U1.24 (A5)
- net GND: now also C1.2, C10.2, C15.1, C16.2, C18.1, C19.1, C2.2, C20.2, C21.2, C22.2, C23.2, C24.1, C25.1, C27.2, C28.1, C36.1, C37.1, C39.1, C4.2, C40.1, C5.2, C6.1, C7.1, C9.2, P1.2, P10.2, P11.2, P12.2, P2.2, P3.2, P4.2, P5.2, P6.2, P9.2, R14.2, R15.2, R17.2, R2.1, R20.2, R24.2, R25.2, U1.29 (GND), U1.4 (GND), U10.3, U11.1, U11.12, U11.5, U12.1, U12.12, U12.5, U13.1 (GND), U14.3 (E), U2.1 (GND), U3.2 (GND), U4.3 (E), U5.1 (GND), U6.4 (GND), U6.7 (EP), U7.4 (GND), U7.7 (EP), U8.3 (E), U9.3 (E); no longer R26.2
- net PIR_IN1: now also U1.8 (D5), U9.1 (C)
- net PIR_Outside: now also U1.25 (A6), U8.1 (C)
- net RFID-Inside-EN: now also R3.1, U1.9 (D6), U6.5 (EN/UVLO)
- net RFID-Outside-EN: now also R4.1, U1.21 (A2), U7.5 (EN/UVLO)
- net Servo_Inside_PWM: now also P4.3, U1.13 (D10)
- net Servo_Outside_PWM: now also P5.3, U1.23 (A4)
- net at R26.1: now also R27.2, U5.7 (DIS)
- new net: C40.2, R30.1, U13.2 (TR), U13.6 (THR)
- new net: R23.1, R24.1, U4.2 (B)
- new net: C17.2, U11.10
- new net: C18.2, C19.2, U11.11
- new net: C21.1, U11.15
- new net: C20.1, U11.16
- new net: R21.2, U11.3
- new net: C11.2, C12.2, C8.2, U11.6
- new net: C13.1, C14.1, C15.2, U11.8
- new net: C17.1, U11.9
- new net: C29.2, C30.2, C31.1, C32.1, C33.1, P8.1
- new net: C31.2, C32.2, C33.2, U12.6
- new net: C37.2, R27.1, U5.2 (TR), U5.6 (THR)
- new net: P11.1, R31.2
- new net: P12.3, R32.2
- new net: C11.1, C12.1, C13.2, C14.2, C8.1, P7.1
- new net: R25.1, R32.1, U14.2 (B)
- new net: R19.1, R20.1, U9.2 (B)
- new net: C3.1, U3.1 (CB)
- new net: R1.1, R2.2, U3.3 (FB)
- new net: C3.2, L1.1, U3.6 (SW)
- new net: R31.1, U13.3 (Q)
- new net: C39.2, U13.5 (CV)
- new net: R29.1, R30.2, U13.7 (DIS)
- new net: P7.2, R21.1
- new net: R17.1, R18.1, U8.2 (B)
- new net: R19.2, U10.2
- new net: R28.1, U5.3 (Q)
- new net: C36.2, U5.5 (CV)
- new net: C28.2, C29.1, C30.1, U12.8
- new net: C23.1, U12.16
- new net: P8.2, R22.1
- new net: R22.2, U12.3
- new net: P10.1, R28.2
- new net: P2.1, R13.2
- new net: C24.2, C25.2, U12.11
- new net: P9.3, R23.2
- new net: C22.1, U12.15
- new net: P6.3, R18.2
- new net: C26.1, U12.9
- new net: C26.2, U12.10
- new net: P3.1, R16.2
- new net RFID-Inside-SHDN: U11.14, U6.1 (VOUT), U6.2 (QOD)
- new net RFID-Outside-SHDN: U12.14, U7.1 (VOUT), U7.2 (QOD)
- new net RFID_Inside_3.3VCLK: Q1.2 (S), R5.1, U1.11 (D8)
- new net RFID_Inside_3.3VDMOD: Q4.2 (S), R12.1, U1.10 (D7)
- new net RFID_Inside_5VCLK: Q1.3 (D), R6.1, U11.2
- new net RFID_Inside_5VDMOD: Q4.3 (D), R11.1, U11.13
- new net RFID_Outside_3.3VCLK: Q2.2 (S), R8.1, U1.6 (D3)
- new net RFID_Outside_3v3VDMOD: Q3.2 (S), R9.1, U1.5 (D2)
- new net RFID_Outside_5VCLK: Q2.3 (D), R7.1, U12.2
- new net RFID_Outside_5VDMOD: Q3.3 (D), R10.1, U12.13
- new net Tunnel_IR_IN: U1.14 (D11), U4.1 (C)
- new net Tunnel_IR_OUT: U1.15 (D12), U14.1 (C)
- no-connect marks 11 -> 15
Other:
- note added: "Controller"
- note added: "Designed for SFH-4546"
- note added: "Designed for TSOP18138/TSOP18338/TSOP18538"
- note added: "Designed for TSOP18156/TSOP18356/TSOP18557"
- note added: "FlapIR inside"
- note added: "FlapIR outside"
- note added: "PIR inside"
- note added: "PIR outside"
- note added: "Power"
- note added: "RFID Inside"
- note added: "RFID Inside sleep"
- note added: "RFID Outside"
- note added: "RFID Outside sleep"
- note added: "RFID inside signal"
- note added: "RFID outside signal"
- note added: "Servo inside"
- note added: "Servo outside"
- note added: "Tunnel IR LED inside 38KHz"
- note added: "Tunnel IR LED outside 56KHz"
- note added: "Tunnel IR Receiver inside 38KHz"
- note added: "Tunnel IR Receiver outside 56KHz"
- note removed: "47 38 21 18 17 10 9 8 7 6 5 GND RST 44 43"
- note removed: "48 3.3V 46 1 2 3 4 11 12 13 14 VBUS 0 GND VIN"
- note removed: "IR Outside"
- note removed: "Power Connector"
- note removed: "Power Section"
- note removed: "Reserved for TX1"
- note removed: "Reserved for TX2"
- note removed: "SensorsEmbedd on PCB"
- title: (none) -> OpenCatFlap
